File: toshiba-64mbit-adapter.kicad_pcb (KiCad board)
At the start: 2 copper layers, 18 x 55 mm, 9 parts, among them U1 TC5364205, U2 W29GL064C, U3 74HCT244, U4 74HCT244, U5 74HCT244, U6 74HCT244, U7 74HCT244, U8 TPS73633DBV

Commit message: WIP changes
Other:
- net class Default removed
